File: pcb/power_supply.sch (EAGLE design)
At the start: 53 parts, among them IC1 AP1507-D5-13, P1 2k, Q1 DIODES_FMMT493ATADIODES_FMMT4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, Q2 DIODES_FMMT493ATADIODES_FMMT4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, Q3 DIODES_FMMT493ATADIODES_FMMT4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, Q4 DIODES_FMMT493ATADIODES_FMMT4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, Q5 DIODES_FMMT493ATADIODES_FMMT4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, Q6 DIODES_FMMT493ATADIODES_FMMT4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, Q7 DIODES_FMMT493ATADIODES_FMMT4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, Q8 DIODES_FMMT493ATADIODES_FMMT4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, U1 LM1085IT-ADJ

Commit message: pcb - board partially updated
Parts:
- removed C10, C9: 22u, rcl:C-EUC1206
- removed L9: HPI1040-220, SRR1050A-151Y:SRR1050A-151Y
- added C3, C4: 100n, rcl:C-EUC0603
- added CON1: +, con-phoenix-254:MPT2
- C7, C8: value 100n -> 22u; device rcl:C-EUC0603 -> rcl:C-EUC1206
- CON2, CON3, CON4, CON5, CON6, CON7, CON8: value 1 -> +
- L1: value 1 -> HPI1040-220; device con-phoenix-254:MPT2 -> SRR1050A-151Y:SRR1050A-151Y
- renumbered L2 to CON2, L3 to CON3, L4 to CON4, L5 to CON5, L6 to CON6, L7 to CON7, L8 to CON8, R100 to R18, R110 to R19, R120 to R20, R90 to R17
Connections:
- removed net N$2 (its old number): ACC1-1.K, SWITCH-2.K
- new net N$4: IC1.FB, R18.2, R19.2
- new net N$7: ACC2-2.K, SWITCH-1.K
- net BAT: now also C3.1, C4.1, SWITCH-2.K; no longer C7.1, C8.1, SWITCH-1.K
- net GND: now also ACC1-1.K, C3.2, C4.2; no longer ACC2-2.K, C10.2, C9.2
- net LIGHTS+: now also CON1-2.1; no longer L1-2.1
- net N$1: now also CON1-1.1; no longer L1-1.1
- net N$32: now also L1.1; no longer L9.1
- net RASP_SUPPLY: now also C7.1, C8.1, L1.2; no longer C10.1, C9.1, IC1.FB, L9.2, R18.2, R19.2
Other:
- moved on the sheet: ACC1-1, ACC1-2, ACC2-1, ACC2-2, C7, C8, SWITCH-1, SWITCH-2

Commit message: pcb - better supply route
Parts:
- RASPBERRY: device RASPBERRY_PI_3_MODEL_B_:RASPBERRY_PI_3_MODEL_B+ -> RASPBERRY_PI_3_MODEL_B_NoScrew:RASPBERRY_PI_3_MODEL_B+
Changed lines of the file:
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@@
 </classes>
 <parts>
-<part name="RASPBERRY" library="RASPBERRY_PI_3_MODEL_B_" deviceset="RASPBERRY_PI_3_MODEL_B+" device=""/>
+<part name="RASPBERRY" library="RASPBERRY_PI_3_MODEL_B_NoScrew" deviceset="RASPBERRY_PI_3_MODEL_B+" device=""/>
 <part name="SUPPLY3" library="supply2" library_urn="urn:adsk.eagle:library:372" deviceset="GND" device=""/>
 <part name="SUPPLY2" library="supply2" library_urn="urn:adsk.eagle:library:372" deviceset="GND" device=""/>
